File: Projects/Full Board/LNA.sch (KiCad schematic (older format))
At the start: 28 parts, among them J1 SMA-J-P-H-ST-EM1, J2 SMA-J-P-H-ST-EM1, J3 Barrel_Jack_MountingPin, Q1 Q_NPN_BEC, U1 BFU790F

Commit message: added full board
Parts:
- removed CC10: 10u, Capacitor_SMD:C_1206_3216Metric, symbol Device:C
- removed CC3, CC4: .47u, Capacitor_SMD:C_0805_2012Metric, symbol Device:C
- removed Csh2: 1.2p, Capacitor_SMD:C_0805_2012Metric, symbol Device:C
- removed J1, J2: SMA-J-P-H-ST-EM1, SAMTEC_SMA-J-P-H-ST-EM1, symbol RandomSMAIFoundOnline:SMA-J-P-H-ST-EM1
- removed J3: Barrel_Jack_MountingPin, Connector_BarrelJack:BarrelJack_Horizontal, symbol Connector:Barrel_Jack_MountingPin
- removed RB2: 9.1k, Resistor_SMD:R_0805_2012Metric, symbol Device:R
- removed RE12, RE13, RE14, RE15: 18, Resistor_SMD:R_0805_2012Metric, symbol Device:R
- removed RFB2: 330, Resistor_SMD:R_0805_2012Metric, symbol Device:R
- added CC_LNA3, CC_LNA4: .47u, Capacitor_SMD:C_0805_2012Metric, symbol Device:C
- added Csh1: 1.2p, Capacitor_SMD:C_0805_2012Metric, symbol Device:C
- added RB1: 9.1k, Resistor_SMD:R_0805_2012Metric, symbol Device:R
- added RE2, RE3, RE4, RE5: 18, Resistor_SMD:R_0805_2012Metric, symbol Device:R
- added RFB4: 330, Resistor_SMD:R_0805_2012Metric, symbol Device:R
- renumbered CC2 to CC_LNA_2, CC1 to CC_LNA_In1, RE21 to RE6, RE22 to RE7, Ri2 to Ri1, Rsh2 to Rsh1, U1 to U_BFQ790
Connections:
- net labels added: +5V, AntennaIn, LNA_Out
- net labels removed: VCC
- wire segments 65 -> 57
- no-connect marks 1 -> 0
