File: Projects/Full Board/DiffToSingle.sch (KiCad schematic (older format))
At the start: 10 parts

Commit message: This is the latest version with updated footprints etc
Parts:
- added JI_Out1, JQ_Out1: 221789-1, TE_221789-1, symbol 221789-1:221789-1
- added L11, L22: 470nH, Inductor_SMD:L_0805_2012Metric, symbol Device:L
Connections:
- net GND: now also JI_Out1.S1 (SHIELD), JI_Out1.S2 (SHIELD), JI_Out1.S3 (SHIELD), JI_Out1.S4 (SHIELD), JQ_Out1.S1 (SHIELD), JQ_Out1.S2 (SHIELD), JQ_Out1.S3 (SHIELD), JQ_Out1.S4 (SHIELD)
- net I_Filter: now also JI_Out1.1 (P1), L11.1; no longer L1.1
- net Q_Filter: now also JQ_Out1.1 (P1), L22.1; no longer L2.1
- new net: L1.1, L11.2
- new net: L2.1, L22.2
Other:
- moved on the sheet: C_Filter2, C_Filter4
Changed lines of the file:
@@
 L Device:C C_Filter2
 U 1 1 60232846
-P 5800 2300
-F 0 "C_Filter2" H 5915 2346 50  0000 L CNN
-F 1 "160pF" H 5915 2255 50  0000 L CNN
-F 2 "Capacitor_SMD:C_0805_2012Metric" H 5838 2150 50  0001 C CNN
-F 3 "~" H 5800 2300 50  0001 C CNN
-	1    5800 2300
+P 6400 2300
+F 0 "C_Filter2" H 6515 2346 50  0000 L CNN
+F 1 "160pF" H 6515 2255 50  0000 L CNN
+F 2 "Capacitor_SMD:C_0805_2012Metric" H 6438 2150 50  0001 C CNN
+F 3 "~" H 6400 2300 50  0001 C CNN
+	1    6400 2300
 	1    0    0    -1
 $EndComp
@@
 	5250 2100 5400 2100
 Wire Wire Line
-	5800 2150 5800 2100
-Wire Wire Line
-	5800 2100 5700 2100
+	6400 2150 6400 2100
 $Comp
 L power:GND #PWR0135
@@
 L power:GND #PWR0136
 U 1 1 602342D8
-P 5800 2500
-F 0 "#PWR0136" H 5800 2250 50  0001 C CNN
-F 1 "GND" H 5805 2327 50  0000 C CNN
-F 2 "" H 5800 2500 50  0001 C CNN
-F 3 "" H 5800 2500 50  0001 C CNN
-	1    5800 2500
+P 6400 2500
+F 0 "#PWR0136" H 6400 2250 50  0001 C CNN
+F 1 "GND" H 6405 2327 50  0000 C CNN
+F 2 "" H 6400 2500 50  0001 C CNN
+F 3 "" H 6400 2500 50  0001 C CNN
+	1    6400 2500
 	1    0    0    -1
 $EndComp
@@
 L Device:C C_Filter4
 U 1 1 60244378
-P 5800 1500
-F 0 "C_Filter4" H 5915 1546 50  0000 L CNN
-F 1 "160pF" H 5915 1455 50  0000 L CNN
-F 2 "Capacitor_SMD:C_0805_2012Metric" H 5838 1350 50  0001 C CNN
-F 3 "~" H 5800 1500 50  0001 C CNN
-	1    5800 1500
+P 6400 1500
+F 0 "C_Filter4" H 6515 1546 50  0000 L CNN
+F 1 "160pF" H 6515 1455 50  0000 L CNN
+F 2 "Capacitor_SMD:C_0805_2012Metric" H 6438 1350 50  0001 C CNN
+F 3 "~" H 6400 1500 50  0001 C CNN
+	1    6400 1500
 	1    0    0    -1
 $EndComp
@@
 	5250 1300 5400 1300
 Wire Wire Line
-	5800 1350 5800 1300
-Wire Wire Line
-	5800 1300 5700 1300
+	6400 1350 6400 1300
 $Comp
 L power:GND #PWR0139
@@
 L power:GND #PWR0140
 U 1 1 60244390
-P 5800 1650
-F 0 "#PWR0140" H 5800 1400 50  0001 C CNN
-F 1 "GND" H 5805 1477 50  0000 C CNN
-F 2 "" H 5800 1650 50  0001 C CNN
-F 3 "" H 5800 1650 50  0001 C CNN
-	1    5800 1650
+P 6400 1650
+F 0 "#PWR0140" H 6400 1400 50  0001 C CNN
+F 1 "GND" H 6405 1477 50  0000 C CNN
+F 2 "" H 6400 1650 50  0001 C CNN
+F 3 "" H 6400 1650 50  0001 C CNN
+	1    6400 1650
 	1    0    0    -1
 $EndComp
@@
 Wire Wire Line
 	4600 1300 5250 1300
-Text Label 6000 1300 0    50   ~ 0
+Text Label 6500 1300 0    50   ~ 0
 Q_Filtered
-Text Label 5950 2100 0    50   ~ 0
+Text Label 6450 2100 0    50   ~ 0
 I_Filtered
 Wire Wire Line
@@
 	2700 2450 2700 2300
 Wire Wire Line
-	5800 2500 5800 2450
+	6400 2500 6400 2450
 Text HLabel 1800 1000 0    50   Input ~ 0
 Q-
@@
 Text HLabel 1800 2450 0    50   Input ~ 0
 I-
-Wire Wire Line
-	5800 1300 6650 1300
-Connection ~ 5800 1300
-Wire Wire Line
-	5800 2100 6650 2100
-Connection ~ 5800 2100
 Text HLabel 6650 2100 2    50   Input ~ 0
 I_Filter
 Text HLabel 6650 1300 2    50   Input ~ 0
 Q_Filter
+Connection ~ 6400 1300
+Wire Wire Line
+	5700 1300 5850 1300
+$Comp
+L Device:L L22
+U 1 1 60232E16
+P 6000 1300
+F 0 "L22" V 5819 1300 50  0000 C CNN
+F 1 "470nH" V 5910 1300 50  0000 C CNN
+F 2 "Inductor_SMD:L_0805_2012Metric" H 6000 1300 50  0001 C CNN
+F 3 "~" H 6000 1300 50  0001 C CNN
+	1    6000 1300
+	0    1    1    0
+$EndComp
+Wire Wire Line
+	6150 1300 6400 1300
+Connection ~ 6400 2100
+Wire Wire Line
+	5700 2100 5850 2100
+$Comp
+L Device:L L11
+U 1 1 602344FE
+P 6000 2100
+F 0 "L11" V 5819 2100 50  0000 C CNN
+F 1 "470nH" V 5910 2100 50  0000 C CNN
+F 2 "Inductor_SMD:L_0805_2012Metric" H 6000 2100 50  0001 C CNN
+F 3 "~" H 6000 2100 50  0001 C CNN
+	1    6000 2100
+	0    1    1    0
+$EndComp
+Wire Wire Line
+	6150 2100 6400 2100
+Wire Wire Line
+	6400 1300 6550 1300
+Wire Wire Line
+	6400 2100 6550 2100
+Wire Wire Line
+	6550 1300 6550 1500
+Connection ~ 6550 1300
+Wire Wire Line
+	6550 1300 6650 1300
+Wire Wire Line
+	6550 2100 6550 2350
+Connection ~ 6550 2100
+Wire Wire Line
+	6550 2100 6650 2100
+$Comp
+L power:GND #PWR0112
+U 1 1 60243E71
+P 7050 2550
+F 0 "#PWR0112" H 7050 2300 50  0001 C CNN
+F 1 "GND" H 7055 2377 50  0000 C CNN
+F 2 "" H 7050 2550 50  0001 C CNN
+F 3 "" H 7050 2550 50  0001 C CNN
+	1    7050 2550
+	1    0    0    -1
+$EndComp
+$Comp
+L power:GND #PWR0113
+U 1 1 60244119
+P 7100 1700
+F 0 "#PWR0113" H 7100 1450 50  0001 C CNN
+F 1 "GND" H 7105 1527 50  0000 C CNN
+F 2 "" H 7100 1700 50  0001 C CNN
+F 3 "" H 7100 1700 50  0001 C CNN
+	1    7100 1700
+	1    0    0    -1
+$EndComp
+$Comp
+L 221789-1:221789-1 JQ_Out1
+U 1 1 60260DDE
+P 7500 1600
+F 0 "JQ_Out1" H 7270 1646 50  0000 R CNN
+F 1 "221789-1" H 7270 1555 50  0000 R CNN
+F 2 "TE_221789-1" H 7500 1600 50  0001 L BNN
+F 3 "" H 7500 1600 50  0001 L BNN
+F 4 "1" H 7500 1600 50  0001 L BNN "Number_of_Positions"
+F 5 "Compliant with Exemptions" H 7500 1600 50  0001 L BNN "EU_RoHS_Compliance"
+F 6 "221789-1" H 7500 1600 50  0001 L BNN "Comment"
+	1    7500 1600
+	-1   0    0    -1
+$EndComp
+Wire Wire Line
+	6550 1500 7100 1500
+$Comp
+L 221789-1:221789-1 JI_Out1
+U 1 1 60264324
+P 7450 2450
+F 0 "JI_Out1" H 7220 2496 50  0000 R CNN
+F 1 "221789-1" H 7220 2405 50  0000 R CNN
+F 2 "TE_221789-1" H 7450 2450 50  0001 L BNN
+F 3 "" H 7450 2450 50  0001 L BNN
+F 4 "1" H 7450 2450 50  0001 L BNN "Number_of_Positions"
+F 5 "Compliant with Exemptions" H 7450 2450 50  0001 L BNN "EU_RoHS_Compliance"
+F 6 "221789-1" H 7450 2450 50  0001 L BNN "Comment"
+	1    7450 2450
+	-1   0    0    -1
+$EndComp
+Wire Wire Line
+	6550 2350 7050 2350
 $EndSCHEMATC
