File: Projects/Full Board/Full Board.kicad_pcb (KiCad board)
At the start: 2 copper layers, 105 parts, among them IC2 MC74ACT86DG, J1 SMA-J-P-H-ST-EM1, J2 SMA-J-P-H-ST-EM1, J3 Conn_01x02, J4 Conn_01x02, J7 Conn_01x04, J8 Conn_01x05, Q1 Q_NPN_BEC, U1 LMV116MF, U2 TLV2374ID, U3 SFECF10M7EA00-R0, U4 SN74ACT04IDREP

Commit message: This is the latest version with updated footprints etc
Parts:
- removed C13, C14, C17, C19: C, Capacitor_SMD:C_0603_1608Metric
- removed L5, L6: L, Inductor_SMD:L_0603_1608Metric
- added JI_Out1: 221789-1, AdditionalLibs:TE_221789-1, F.Cu at (145.8, 72.6)
- added JQ_Out1: 221789-1, AdditionalLibs:TE_221789-1, F.Cu at (163.1, 71.6)
- added L11: 470nH, Inductor_SMD:L_0805_2012Metric, F.Cu at (150.4, 81.8)
- added L22: 470nH, Inductor_SMD:L_0805_2012Metric, F.Cu at (157.5, 81.8)
- C16, C21, C22, C29, C30, CC1, C_CMG1, Cin1, R1, R2: moved to B.Cu
- moved J_Out1 112.3 mm to (105.7, 55.1), turned to 180 degrees
- moved Cin1 106.7 mm to (105.3, 97.0), turned to 180 degrees
- moved R2 105.0 mm to (108.1, 94.4), turned to 90 degrees
- moved C_CMG1 95.3 mm to (115.2, 95.9), turned to 270 degrees
- moved U_TRF1 95.2 mm to (134.4, 90.2)
- moved CC2 95.2 mm to (125.2, 90.4)
- moved CRF1 95.2 mm to (130.3, 98.6)
- moved LRF1 95.2 mm to (129.3, 91.5)
- moved R_Pullup2 95.2 mm to (120.9, 87.5)
- moved CDC1 95.2 mm to (135.4, 94.2)
- moved CRF2 95.2 mm to (130.2, 95.2)
- moved R_Pullup1 95.2 mm to (120.9, 93.7)
- moved Rout1 95.1 mm to (105.4, 84.4), turned to 270 degrees
- moved IC2 95.1 mm to (104.1, 91.7), turned to 270 degrees
- moved R_CMG1 93.5 mm to (111.6, 96.4), turned to 180 degrees
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Connections:
- net Net-(Cin1-Pad1) renamed /IF_FilterAndAmp/InputToTLV
- L1 pad 1: /SummerAndAmp/I -> Net-(L1-Pad1)
- L2 pad 1: /SummerAndAmp/Q -> Net-(L2-Pad1)
Routing:
- net +5V: track 1.11 -> 52.1 mm, vias 1 -> 14
- net /SummerAndAmp/Q: track 8.78 -> 49.7 mm
- net 3.3V: track 3.70 -> 41.9 mm, vias 0 -> 2
- net /SummerAndAmp/I: track 8.78 -> 43.1 mm
- net /IF_FilterAndAmp/AudioSignalOut: track 0.00 -> 30.1 mm
- net /IF_FilterAndAmp/CMG: track 0.00 -> 17.8 mm, vias 0 -> 1
- net /DiffToSingle/Q-: track 3.89 -> 19.2 mm
- net -5V: track 0.00 -> 14.1 mm, vias 0 -> 1
- net /IF_FilterAndAmp/FilteredIF: track 0.00 -> 13.3 mm
- net /DiffToSingle/Q+: track 3.84 -> 17.1 mm
- net /IF_FilterAndAmp/InputToTLV: track 0.00 -> 12.0 mm, vias 0 -> 1
- net /IF_FilterAndAmp/IF_Lim: track 0.00 -> 10.1 mm
- net /Mixer/LO_In: track 17.8 -> 8.11 mm
- net /DiffToSingle/I+: track 4.06 -> 13.0 mm
- net /IF_FilterAndAmp/4Y: track 0.00 -> 8.65 mm
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- added copper zone on In2.Cu, net +5V
- added copper zone on B.Cu, net GND
- added copper zone on F.Cu, net GND
- added copper zone on In1.Cu, net GND
Other:
- board outline added: 113 x 70.1 mm
- copper layers 2 -> 4
- board text added: "+5V"
- board text added: "-5V"
- board text added: "3.3V"
- board text added: "GND"
