File: Projects/Full Board/IF_FilterAndAmp.sch (KiCad schematic (older format))
At the start: 27 parts, among them IC2 MC74ACT86DG, U2 TLV2374ID, U3 SFECF10M7EA00-R0, U4 SN74ACT04IDREP

Commit message: This is the latest version with updated footprints etc
Connections:
- net InputToTLV: now reaches Cin1.1, R1.2, R2.1, U2.3 (1IN+)
Changed lines of the file:
@@
 	0    1    1    0
 $EndComp
+Text Label 1200 4100 0    50   ~ 0
+InputToTLV
 $EndSCHEMATC
