File: Projects/DemoProject/DemoProject.kicad_pcb (KiCad board)
At the start: 2 copper layers, 28.7 x 18 mm, 5 parts, among them J1 4P2C, J2 4P2C, U1 LMC358

Commit message: This is the latest version with updated footprints etc
Routing:
- net GND: vias 1 -> 28
