File: Projects/DemodulatorCircuit/DemodulatorCircuit.sch (KiCad schematic (older format))
At the start: 22 parts, among them IC2 MC74ACT86DG, J1 SMA-J-P-H-ST-EM1, J2 Conn_01x02, J3 SMA-J-P-H-ST-EM1, U1 TLV3501AID, U2 TLV2374ID, U3 SFECF10M7EA00-R0, U4 SN74ACT04IDREP

Commit message: This is the latest version with updated footprints etc
Parts:
- added C_Inv_1, C_Inv_2, C_Inv_3, C_Inv_4, C_Inv_5: 8.2pF, Capacitor_SMD:C_0603_1608Metric, symbol Device:C
- added R_Inv_1, R_Inv_2, R_Inv_3, R_Inv_4, R_Inv_5: 1k, Resistor_SMD:R_0603_1608Metric, symbol Device:R
Connections:
- net 1Y: now also C_Inv_1.1, R_Inv_1.1; no longer U4.3 (2A)
- net 2Y: now also C_Inv_2.1, R_Inv_2.1; no longer U4.5 (3A)
- net 3Y: now also C_Inv_3.1, R_Inv_3.1; no longer U4.9 (4A)
- net 4Y: now also C_Inv_4.1, R_Inv_4.1; no longer U4.11 (5A)
- net 5Y: now also C_Inv_5.1, R_Inv_5.1; no longer U4.13 (6A)
- net GND: now also C_Inv_1.2, C_Inv_2.2, C_Inv_3.2, C_Inv_4.2, C_Inv_5.2
- new net: R_Inv_1.2, U4.3 (2A)
- new net: R_Inv_2.2, U4.5 (3A)
- new net: R_Inv_3.2, U4.9 (4A)
- new net: R_Inv_4.2, U4.11 (5A)
- new net: R_Inv_5.2, U4.13 (6A)
Other:
- moved on the sheet: U4

Commit message: post board review they are all ready to order
Connections:
- net 3Y: now also C_Inv_5.1, R_Inv_5.1; no longer C_Inv_3.1, R_Inv_3.1
- net 4Y: now also IC2.2 (INPUT_1_2); no longer C_Inv_4.1, R_Inv_4.1
- net 5Y: now also C_Inv_3.1, R_Inv_3.1; no longer C_Inv_5.1, R_Inv_5.1
- net IFQ_LIM renamed 6Y
- net 6Y: now also C_Inv_4.1, R_Inv_4.1; no longer IC2.2 (INPUT_1_2)
Changed lines of the file:
@@
 	1650 1600 2250 1600
-$Comp
-L SN74ACT04IDREP:SN74ACT04IDREP U4
-U 1 1 602C3E51
-P 8150 4450
-F 0 "U4" H 8150 5220 50  0000 C CNN
-F 1 "SN74ACT04IDREP" H 8150 5129 50  0000 C CNN
-F 2 "SOIC127P600X175-14N" H 8150 4450 50  0001 L BNN
-F 3 "" H 8150 4450 50  0001 L BNN
-	1    8150 4450
-	0    1    1    0
-$EndComp
 $Comp
 L MC74ACT86DG:MC74ACT86DG IC2
@@
 	8250 5150 8250 5350
 Wire Wire Line
-	8150 5150 8150 5350
-Wire Wire Line
 	8050 5150 8050 5350
 Wire Wire Line
@@
 Wire Wire Line
 	9150 4450 9150 6350
-Wire Wire Line
-	9150 6350 7950 6350
-Wire Wire Line
-	7950 5150 7950 6350
 Connection ~ 9150 4450
 Wire Wire Line
@@
 	8150 3550 8150 3750
 Text Label 8150 2900 0    50   ~ 0
-3Y
+5Y
 $Comp
 L Device:R R_Inv_3
@@
 	8050 3550 8050 3750
 Text Label 8050 2900 0    50   ~ 0
-4Y
+6Y
 $Comp
 L Device:R R_Inv_4
@@
 	7950 3550 7950 3750
 Text Label 7950 2900 0    50   ~ 0
-5Y
+3Y
 $Comp
 L Device:R R_Inv_5
@@
 Wire Wire Line
 	9400 2050 9600 2050
+$Comp
+L SN74ACT04IDREP:SN74ACT04IDREP U4
+U 1 1 602C3E51
+P 8150 4450
+F 0 "U4" H 8150 5220 50  0000 C CNN
+F 1 "SN74ACT04IDREP" H 8150 5129 50  0000 C CNN
+F 2 "SOIC127P600X175-14N" H 8150 4450 50  0001 L BNN
+F 3 "" H 8150 4450 50  0001 L BNN
+	1    8150 4450
+	0    1    1    0
+$EndComp
+Text Label 7950 5350 0    50   ~ 0
+6Y
+Wire Wire Line
+	7950 5150 7950 5350
+Wire Wire Line
+	8150 5150 8150 6350
+Wire Wire Line
+	8150 6350 9150 6350
 $EndSCHEMATC
