File: Projects/LNA2/LNA2.sch (KiCad schematic (older format))
At the start: 14 parts, among them J1 SMA-J-P-H-ST-EM1, J2 SMA-J-P-H-ST-EM1, J3 Barrel_Jack_MountingPin, U1 TRF37A73, U2 TPS7A0533PDBV

Commit message: Created a new file
Parts:
- CC3: footprint Capacitor_SMD:C_0805_2012Metric -> Capacitor_SMD:C_1206_3216Metric
Other:
- moved on the sheet: CC3, J3
Changed lines of the file:
@@
 L Connector:Barrel_Jack_MountingPin J3
 U 1 1 6010B5E5
-P 1350 1450
-F 0 "J3" H 1407 1767 50  0000 C CNN
-F 1 "Barrel_Jack_MountingPin" H 1407 1676 50  0000 C CNN
-F 2 "Connector_BarrelJack:BarrelJack_Horizontal" H 1400 1410 50  0001 C CNN
-F 3 "~" H 1400 1410 50  0001 C CNN
-	1    1350 1450
+P 2650 1450
+F 0 "J3" H 2707 1767 50  0000 C CNN
+F 1 "Barrel_Jack_MountingPin" H 2707 1676 50  0000 C CNN
+F 2 "Connector_BarrelJack:BarrelJack_Horizontal" H 2700 1410 50  0001 C CNN
+F 3 "~" H 2700 1410 50  0001 C CNN
+	1    2650 1450
 	1    0    0    -1
 $EndComp
-NoConn ~ 1350 1750
+NoConn ~ 2650 1750
 $Comp
 L power:VCC #PWR0107
 U 1 1 6010C0C3
-P 2100 1100
-F 0 "#PWR0107" H 2100 950 50  0001 C CNN
-F 1 "VCC" H 2115 1273 50  0000 C CNN
-F 2 "" H 2100 1100 50  0001 C CNN
-F 3 "" H 2100 1100 50  0001 C CNN
-	1    2100 1100
+P 3400 1100
+F 0 "#PWR0107" H 3400 950 50  0001 C CNN
+F 1 "VCC" H 3415 1273 50  0000 C CNN
+F 2 "" H 3400 1100 50  0001 C CNN
+F 3 "" H 3400 1100 50  0001 C CNN
+	1    3400 1100
 	1    0    0    -1
 $EndComp
@@
 L Device:C CC3
 U 1 1 6010D31A
-P 2100 1450
-F 0 "CC3" V 1848 1450 50  0000 C CNN
-F 1 "10u" V 1939 1450 50  0000 C CNN
-F 2 "Capacitor_SMD:C_0805_2012Metric" H 2138 1300 50  0001 C CNN
-F 3 "~" H 2100 1450 50  0001 C CNN
-	1    2100 1450
+P 3400 1450
+F 0 "CC3" V 3148 1450 50  0000 C CNN
+F 1 "10u" V 3239 1450 50  0000 C CNN
+F 2 "Capacitor_SMD:C_1206_3216Metric" H 3438 1300 50  0001 C CNN
+F 3 "~" H 3400 1450 50  0001 C CNN
+	1    3400 1450
 	-1   0    0    1
 $EndComp
 Wire Wire Line
-	1650 1350 1900 1350
+	2950 1350 3200 1350
 Wire Wire Line
-	1900 1350 1900 1250
+	3200 1350 3200 1250
 Wire Wire Line
-	1900 1250 2100 1250
+	3200 1250 3400 1250
 Wire Wire Line
-	2100 1250 2100 1300
+	3400 1250 3400 1300
 Wire Wire Line
-	2100 1100 2100 1250
-Connection ~ 2100 1250
+	3400 1100 3400 1250
+Connection ~ 3400 1250
 Wire Wire Line
-	1900 1550 1900 1750
+	3200 1550 3200 1750
 Wire Wire Line
-	1900 1750 2100 1750
+	3200 1750 3400 1750
 Wire Wire Line
-	2100 1750 2100 1600
+	3400 1750 3400 1600
 Wire Wire Line
-	1650 1550 1900 1550
+	2950 1550 3200 1550
 $Comp
 L power:GND #PWR0108
 U 1 1 6010F8E1
-P 2100 1750
-F 0 "#PWR0108" H 2100 1500 50  0001 C CNN
-F 1 "GND" H 2105 1577 50  0000 C CNN
-F 2 "" H 2100 1750 50  0001 C CNN
-F 3 "" H 2100 1750 50  0001 C CNN
-	1    2100 1750
+P 3400 1750
+F 0 "#PWR0108" H 3400 1500 50  0001 C CNN
+F 1 "GND" H 3405 1577 50  0000 C CNN
+F 2 "" H 3400 1750 50  0001 C CNN
+F 3 "" H 3400 1750 50  0001 C CNN
+	1    3400 1750
 	1    0    0    -1
 $EndComp
-Connection ~ 2100 1750
+Connection ~ 3400 1750
 $Comp
 L Regulator_Linear:TPS7A0533PDBV U2
@@
 	4400 1450 4450 1450
 Wire Wire Line
-	2100 1250 3900 1250
-Wire Wire Line
 	4400 1250 4400 1350
 Connection ~ 4400 1350
@@
 	-1   0    0    1
 $EndComp
-Connection ~ 3900 1250
-Wire Wire Line
-	3900 1250 4400 1250
 $Comp
 L power:GND #PWR0110
@@
 $EndComp
 Connection ~ 5150 1350
-Connection ~ 5200 1350
-Wire Wire Line
-	5200 1350 5150 1350
 Wire Wire Line
 	5150 1350 5450 1350
+Wire Wire Line
+	3400 1250 3900 1250
+Connection ~ 3900 1250
+Wire Wire Line
+	3900 1250 4400 1250
 $EndSCHEMATC

Commit message: post board review they are all ready to order
Parts:
- CC3: footprint Capacitor_SMD:C_1206_3216Metric -> Capacitor_Tantalum_SMD:CP_EIA-6032-28_Kemet-C
Changed lines of the file:
@@
 F 0 "CC3" V 3148 1450 50  0000 C CNN
 F 1 "10u" V 3239 1450 50  0000 C CNN
-F 2 "Capacitor_SMD:C_1206_3216Metric" H 3438 1300 50  0001 C CNN
+F 2 "Capacitor_Tantalum_SMD:CP_EIA-6032-28_Kemet-C" H 3438 1300 50  0001 C CNN
 F 3 "~" H 3400 1450 50  0001 C CNN
 	1    3400 1450
