File: Projects/NJR_Demod/NJR_Demod.kicad_pcb (KiCad board)
At the start: 2 copper layers, 45.7 x 40.6 mm, 17 parts, among them T1 TC1-1-13M+, U1 NJM14570RB1-TE1

Commit message: most up to date
Routing:
- net GND: vias 145 -> 155
