File: Projects/InverterChargePump/InverterChargePump.kicad_pcb (KiCad board)
At the start: 2 copper layers, 76.2 x 76.2 mm, 9 parts, among them U1 LTC1983ES6-5#TRPBF

Commit message: new
Routing:
- net +5V: track 1.27 -> 5.14 mm
