File: Projects/PowerDetector/PowerDetector.kicad_pcb (KiCad board)
At the start: 2 copper layers, 25.4 x 38.7 mm, 23 parts, among them J1 SMA-J-P-H-ST-EM1, J2 Conn_01x03, J4 Conn_01x02, U1 LTC5507, U2 LMV116MF, U3 LMV116MF

Commit message: new
Parts:
- C2: value C -> .47u
Connections:
- RFB3 pad 2: GND -> VCC
Routing:
- net VCC: track 31.9 -> 35.0 mm
- net GND: vias 49 -> 48
