File: Projects/PowerDetector/PowerDetector.sch (KiCad schematic (older format))
At the start: 23 parts, among them J1 SMA-J-P-H-ST-EM1, J2 Conn_01x03, J4 Conn_01x02, U1 LTC5507, U2 LMV116MF, U3 LMV116MF

Commit message: new
Parts:
- C2: value C -> .47u
Connections:
- net GND: no longer RFB3.2
- net VCC: now also RFB3.2
Changed lines of the file:
@@
 P 3200 2125
 F 0 "C2" H 3315 2171 50  0000 L CNN
-F 1 "C" H 3315 2080 50  0000 L CNN
+F 1 ".47u" H 3315 2080 50  0000 L CNN
 F 2 "Capacitor_SMD:C_0805_2012Metric" H 3238 1975 50  0001 C CNN
 F 3 "~" H 3200 2125 50  0001 C CNN
@@
 	8075 2075 7600 2075
 $Comp
-L power:GND #PWR0112
-U 1 1 6054C1B4
-P 5950 3100
-F 0 "#PWR0112" H 5950 2850 50  0001 C CNN
-F 1 "GND" H 5955 2927 50  0000 C CNN
-F 2 "" H 5950 3100 50  0001 C CNN
-F 3 "" H 5950 3100 50  0001 C CNN
-	1    5950 3100
-	1    0    0    -1
-$EndComp
-$Comp
 L power:VEE #PWR0113
 U 1 1 6054C96F
@@
 Wire Wire Line
 	3300 1700 3325 1700
+$Comp
+L power:VCC #PWR?
+U 1 1 6052CEF4
+P 5950 3100
+F 0 "#PWR?" H 5950 2950 50  0001 C CNN
+F 1 "VCC" H 5965 3273 50  0000 C CNN
+F 2 "" H 5950 3100 50  0001 C CNN
+F 3 "" H 5950 3100 50  0001 C CNN
+	1    5950 3100
+	0    1    1    0
+$EndComp
 $EndSCHEMATC
