File: Projects/VVA_Macom/VVA_Macom.kicad_pcb (KiCad board)
At the start: 2 copper layers, 27.9 x 20.3 mm, 7 parts, among them U1 MAAVSS0006TR-3000

Commit message: new
Parts:
- CC3: value 10u -> .47u; footprint Capacitor_Tantalum_SMD:CP_EIA-6032-28_Kemet-C -> Capacitor_SMD:C_0805_2012Metric
- moved CC3 1.69 mm to (142.9, 77.3)
