File: Projects/VVA_Macom/VVA_Macom.sch (KiCad schematic (older format))
At the start: 7 parts, among them U1 MAAVSS0006TR-3000

Commit message: new
Parts:
- removed CC3: 10u, Capacitor_Tantalum_SMD:CP_EIA-6032-28_Kemet-C, symbol Device:CP
- added CC3: .47u, Capacitor_SMD:C_0805_2012Metric, symbol Device:C
Connections:
- net GND: now also CC3.1
- net at JPower1.1 (Pin_1), U1.5 (Vc): now also CC3.2
Changed lines of the file:
@@
 $EndComp
-Wire Wire Line
-	5275 2525 5275 2625
 Wire Wire Line
 	5275 2800 5200 2800
@@
 	4825 3450 5200 3450
 $Comp
-L Device:CP CC3
-U 1 1 604ACBFC
-P 5125 2625
-F 0 "CC3" H 5243 2671 50  0000 L CNN
-F 1 "10u" H 5243 2580 50  0000 L CNN
-F 2 "Capacitor_Tantalum_SMD:CP_EIA-6032-28_Kemet-C" H 5163 2475 50  0001 C CNN
-F 3 "~" H 5125 2625 50  0001 C CNN
-	1    5125 2625
-	0    -1   -1   0
-$EndComp
-Connection ~ 5275 2625
-Wire Wire Line
-	5275 2625 5275 2800
-$Comp
 L power:GND #PWR?
 U 1 1 604AEFDD
@@
 	0    1    1    0
 $EndComp
+Wire Wire Line
+	5275 2525 5275 2625
+$Comp
+L Device:C CC3
+U 1 1 6052A3AA
+P 5125 2625
+F 0 "CC3" V 5377 2625 50  0000 C CNN
+F 1 ".47u" V 5286 2625 50  0000 C CNN
+F 2 "Capacitor_SMD:C_0805_2012Metric" H 5163 2475 50  0001 C CNN
+F 3 "~" H 5125 2625 50  0001 C CNN
+	1    5125 2625
+	0    -1   -1   0
+$EndComp
+Connection ~ 5275 2625
+Wire Wire Line
+	5275 2625 5275 2800
 $EndSCHEMATC
