File: Projects/LNA_1/LNA_1.sch (KiCad schematic (older format))
At the start: 28 parts, among them J1 SMA-J-P-H-ST-EM1, J2 SMA-J-P-H-ST-EM1, J3 Barrel_Jack_MountingPin, Q1 Q_NPN_BEC, U1 BFU790F

Commit message: post board review they are all ready to order
Parts:
- CC10: footprint Capacitor_SMD:C_1206_3216Metric -> Capacitor_Tantalum_SMD:CP_EIA-6032-28_Kemet-C
Changed lines of the file:
@@
 F 0 "CC10" H 2450 1550 50  0000 L CNN
 F 1 "10u" H 2450 1450 50  0000 L CNN
-F 2 "Capacitor_SMD:C_1206_3216Metric" H 2738 1350 50  0001 C CNN
+F 2 "Capacitor_Tantalum_SMD:CP_EIA-6032-28_Kemet-C" H 2738 1350 50  0001 C CNN
 F 3 "~" H 2700 1500 50  0001 C CNN
 	1    2700 1500

Commit message: from my laptop
Parts:
- CC1, CC10, CC2, CC3, CC4, CC5, Csh2: symbol Device:C -> LNA_1-rescue:C-Device
- J1, J2: symbol RandomSMAIFoundOnline:SMA-J-P-H-ST-EM1 -> LNA_1-rescue:SMA-J-P-H-ST-EM1-RandomSMAIFoundOnline
- J3: symbol Connector:Barrel_Jack_MountingPin -> LNA_1-rescue:Barrel_Jack_MountingPin-Connector
- LFB1: symbol Device:L -> LNA_1-rescue:L-Device
- Q1: symbol Device:Q_NPN_BEC -> LNA_1-rescue:Q_NPN_BEC-Device
- RB1A1, RB2, RC1, RE1, RE12, RE13, RE14, RE15, RE21, RE22, RFB1, RFB2, Ri2, Ro1, Rsh2: symbol Device:R -> LNA_1-rescue:R-Device
- U1: symbol AdditionalParts:BFU790F -> LNA_1-rescue:BFU790F-AdditionalParts
Changed lines of the file:
@@
 $EndDescr
 $Comp
-L Device:R RB1A1
+L LNA_1-rescue:R-Device RB1A1
 U 1 1 6006F81B
 P 3300 2300
@@
 $EndComp
 $Comp
-L Device:C CC2
+L LNA_1-rescue:C-Device CC2
 U 1 1 60075EB6
 P 4000 3350
@@
 $EndComp
 $Comp
-L Device:C CC1
+L LNA_1-rescue:C-Device CC1
 U 1 1 600770B4
 P 2850 3850
@@
 $EndComp
 $Comp
-L Device:R RFB1
+L LNA_1-rescue:R-Device RFB1
 U 1 1 60078033
 P 4000 2750
@@
 $EndComp
 $Comp
-L Device:L LFB1
+L LNA_1-rescue:L-Device LFB1
 U 1 1 6007853D
 P 4700 2450
@@
 	4000 2450 4550 2450
 $Comp
-L Device:R RFB2
+L LNA_1-rescue:R-Device RFB2
 U 1 1 6007A24B
 P 5200 2450
@@
 	4850 2450 5050 2450
 $Comp
-L AdditionalParts:BFU790F U1
+L LNA_1-rescue:BFU790F-AdditionalParts U1
 U 1 1 6008C937
 P 4600 3900
@@
 	5600 2450 5350 2450
 $Comp
-L Device:R RE1
+L LNA_1-rescue:R-Device RE1
 U 1 1 600967BC
 P 4350 4900
@@
 $EndComp
 $Comp
-L Device:R RE12
+L LNA_1-rescue:R-Device RE12
 U 1 1 600974A1
 P 4700 4900
@@
 $EndComp
 $Comp
-L Device:R RE13
+L LNA_1-rescue:R-Device RE13
 U 1 1 60097625
 P 5050 4900
@@
 	4700 5050 5050 5050
 $Comp
-L Device:R RE14
+L LNA_1-rescue:R-Device RE14
 U 1 1 60098B6D
 P 5400 4900
@@
 $EndComp
 $Comp
-L Device:R RE15
+L LNA_1-rescue:R-Device RE15
 U 1 1 60098B73
 P 5750 4900
@@
 	3300 3850 4000 3850
 $Comp
-L Device:R RC1
+L LNA_1-rescue:R-Device RC1
 U 1 1 6009E84F
 P 5600 1800
@@
 Connection ~ 5600 2450
 $Comp
-L Device:C CC3
+L LNA_1-rescue:C-Device CC3
 U 1 1 600A01A8
 P 6100 2450
@@
 	5600 1450 5600 1650
 $Comp
-L power:VCC #PWR0102
+L LNA_1-rescue:VCC-power #PWR0102
 U 1 1 600A14F0
 P 3300 1300
@@
 	2200 3850 2700 3850
 $Comp
-L power:GND #PWR0103
+L LNA_1-rescue:GND-power #PWR0103
 U 1 1 600B27E1
 P 2200 3950
@@
 $EndComp
 $Comp
-L power:GND #PWR0104
+L LNA_1-rescue:GND-power #PWR0104
 U 1 1 600BF42B
 P 10000 2850
@@
 $EndComp
 $Comp
-L Device:C CC4
+L LNA_1-rescue:C-Device CC4
 U 1 1 600C2E6D
 P 8400 1450
@@
 $EndComp
 $Comp
-L Device:R RB2
+L LNA_1-rescue:R-Device RB2
 U 1 1 600C3923
 P 6750 1800
@@
 Connection ~ 6750 1450
 $Comp
-L Device:R Ri2
+L LNA_1-rescue:R-Device Ri2
 U 1 1 600CB60C
 P 7050 2450
@@
 	6750 2450 6900 2450
 $Comp
-L Device:R Rsh2
+L LNA_1-rescue:R-Device Rsh2
 U 1 1 600CEABE
 P 7500 2700
@@
 	7500 2450 7500 2550
 $Comp
-L Device:C Csh2
+L LNA_1-rescue:C-Device Csh2
 U 1 1 600D073B
 P 7500 3250
@@
 	8200 1450 8250 1450
 $Comp
-L power:GND #PWR0105
+L LNA_1-rescue:GND-power #PWR0105
 U 1 1 600CFB84
 P 7500 3550
@@
 $EndComp
 $Comp
-L power:GND #PWR0106
+L LNA_1-rescue:GND-power #PWR0106
 U 1 1 600DD319
 P 8650 1550
@@
 	8650 1450 8650 1550
 $Comp
-L Device:R RE21
+L LNA_1-rescue:R-Device RE21
 U 1 1 600DE571
 P 8100 3250
@@
 $EndComp
 $Comp
-L Device:R RE22
+L LNA_1-rescue:R-Device RE22
 U 1 1 600DF60E
 P 8500 3250
@@
 Connection ~ 8200 3100
 $Comp
-L Device:R Ro1
+L LNA_1-rescue:R-Device Ro1
 U 1 1 600E443C
 P 9000 2750
@@
 $EndComp
 $Comp
-L Device:C CC5
+L LNA_1-rescue:C-Device CC5
 U 1 1 600E4BF9
 P 9450 2750
@@
 	5050 5150 5050 5050
 $Comp
-L power:GND #PWR0101
+L LNA_1-rescue:GND-power #PWR0101
 U 1 1 600A0F24
 P 5050 5150
@@
 $EndComp
 $Comp
-L power:GND #PWR0107
+L LNA_1-rescue:GND-power #PWR0107
 U 1 1 600A2687
 P 8300 3500
@@
 $EndComp
 $Comp
-L power:VCC #PWR0108
+L LNA_1-rescue:VCC-power #PWR0108
 U 1 1 600FAC3B
 P 2700 1350
@@
 $EndComp
 $Comp
-L power:GND #PWR0109
+L LNA_1-rescue:GND-power #PWR0109
 U 1 1 600FB0E8
 P 2700 1800
@@
 $EndComp
 $Comp
-L Connector:Barrel_Jack_MountingPin J3
+L LNA_1-rescue:Barrel_Jack_MountingPin-Connector J3
 U 1 1 60111861
 P 1950 1500
@@
 NoConn ~ 2250 1800
 $Comp
-L RandomSMAIFoundOnline:SMA-J-P-H-ST-EM1 J1
+L LNA_1-rescue:SMA-J-P-H-ST-EM1-RandomSMAIFoundOnline J1
 U 1 1 60135EC5
 P 2100 3950
@@
 $EndComp
 $Comp
-L Device:Q_NPN_BEC Q1
+L LNA_1-rescue:Q_NPN_BEC-Device Q1
 U 1 1 60109097
 P 8100 2450
@@
 	2600 1350 2700 1350
 $Comp
-L Device:C CC10
+L LNA_1-rescue:C-Device CC10
 U 1 1 6010E877
 P 2700 1500
@@
 Connection ~ 2700 1650
 $Comp
-L RandomSMAIFoundOnline:SMA-J-P-H-ST-EM1 J2
+L LNA_1-rescue:SMA-J-P-H-ST-EM1-RandomSMAIFoundOnline J2
 U 1 1 6013753B
 P 10100 2850

Commit message: last update
Parts:
- removed J3: Barrel_Jack_MountingPin, Connector_BarrelJack:BarrelJack_Horizontal, symbol LNA_1-rescue:Barrel_Jack_MountingPin-Connector
- added J3: Conn_01x02, Connector_PinSocket_2.00mm:PinSocket_1x02_P2.00mm_Vertical, symbol Connector_Generic:Conn_01x02
- CC1, CC2, CC3, CC4, CC5, Csh2: footprint Capacitor_SMD:C_0805_2012Metric -> Capacitor_SMD:C_0603_1608Metric
- LFB1: footprint Inductor_SMD:L_0805_2012Metric -> Inductor_SMD:L_0603_1608Metric
- RB1A1, RB2, RC1, RE1, RE12, RE13, RE14, RE15, RE21, RE22, RFB1, RFB2, Ri2, Ro1, Rsh2: footprint Resistor_SMD:R_0805_2012Metric -> Resistor_SMD:R_0603_1608Metric
Connections:
- net GND: now also J3.2 (Pin_2)
- net VCC: now also J3.1 (Pin_1)
- no-connect marks 1 -> 0
Changed lines of the file:
@@
 F 0 "RB1A1" H 3230 2254 50  0000 R CNN
 F 1 "47k" H 3230 2345 50  0000 R CNN
-F 2 "Resistor_SMD:R_0805_2012Metric" V 3230 2300 50  0001 C CNN
+F 2 "Resistor_SMD:R_0603_1608Metric" V 3230 2300 50  0001 C CNN
 F 3 "~" H 3300 2300 50  0001 C CNN
 	1    3300 2300
@@
 F 0 "CC2" H 4115 3396 50  0000 L CNN
 F 1 ".47u" H 4115 3305 50  0000 L CNN
-F 2 "Capacitor_SMD:C_0805_2012Metric" H 4038 3200 50  0001 C CNN
+F 2 "Capacitor_SMD:C_0603_1608Metric" H 4038 3200 50  0001 C CNN
 F 3 "~" H 4000 3350 50  0001 C CNN
 	1    4000 3350
@@
 F 0 "CC1" H 2965 3896 50  0000 L CNN
 F 1 ".47u" H 2965 3805 50  0000 L CNN
-F 2 "Capacitor_SMD:C_0805_2012Metric" H 2888 3700 50  0001 C CNN
+F 2 "Capacitor_SMD:C_0603_1608Metric" H 2888 3700 50  0001 C CNN
 F 3 "~" H 2850 3850 50  0001 C CNN
 	1    2850 3850
@@
 F 0 "RFB1" H 3930 2704 50  0000 R CNN
 F 1 "330" H 3930 2795 50  0000 R CNN
-F 2 "Resistor_SMD:R_0805_2012Metric" V 3930 2750 50  0001 C CNN
+F 2 "Resistor_SMD:R_0603_1608Metric" V 3930 2750 50  0001 C CNN
 F 3 "~" H 4000 2750 50  0001 C CNN
 	1    4000 2750
@@
 F 0 "LFB1" V 4519 2450 50  0000 C CNN
 F 1 "130n" V 4610 2450 50  0000 C CNN
-F 2 "Inductor_SMD:L_0805_2012Metric" H 4700 2450 50  0001 C CNN
+F 2 "Inductor_SMD:L_0603_1608Metric" H 4700 2450 50  0001 C CNN
 F 3 "~" H 4700 2450 50  0001 C CNN
 	1    4700 2450
@@
 F 0 "RFB2" V 5407 2450 50  0000 C CNN
 F 1 "330" V 5316 2450 50  0000 C CNN
-F 2 "Resistor_SMD:R_0805_2012Metric" V 5130 2450 50  0001 C CNN
+F 2 "Resistor_SMD:R_0603_1608Metric" V 5130 2450 50  0001 C CNN
 F 3 "~" H 5200 2450 50  0001 C CNN
 	1    5200 2450
@@
 F 0 "RE1" H 4280 4854 50  0000 R CNN
 F 1 "18" H 4280 4945 50  0000 R CNN
-F 2 "Resistor_SMD:R_0805_2012Metric" V 4280 4900 50  0001 C CNN
+F 2 "Resistor_SMD:R_0603_1608Metric" V 4280 4900 50  0001 C CNN
 F 3 "~" H 4350 4900 50  0001 C CNN
 	1    4350 4900
@@
 F 0 "RE12" H 4630 4854 50  0000 R CNN
 F 1 "18" H 4630 4945 50  0000 R CNN
-F 2 "Resistor_SMD:R_0805_2012Metric" V 4630 4900 50  0001 C CNN
+F 2 "Resistor_SMD:R_0603_1608Metric" V 4630 4900 50  0001 C CNN
 F 3 "~" H 4700 4900 50  0001 C CNN
 	1    4700 4900
@@
 F 0 "RE13" H 4980 4854 50  0000 R CNN
 F 1 "18" H 4980 4945 50  0000 R CNN
-F 2 "Resistor_SMD:R_0805_2012Metric" V 4980 4900 50  0001 C CNN
+F 2 "Resistor_SMD:R_0603_1608Metric" V 4980 4900 50  0001 C CNN
 F 3 "~" H 5050 4900 50  0001 C CNN
 	1    5050 4900
@@
 F 0 "RE14" H 5330 4854 50  0000 R CNN
 F 1 "18" H 5330 4945 50  0000 R CNN
-F 2 "Resistor_SMD:R_0805_2012Metric" V 5330 4900 50  0001 C CNN
+F 2 "Resistor_SMD:R_0603_1608Metric" V 5330 4900 50  0001 C CNN
 F 3 "~" H 5400 4900 50  0001 C CNN
 	1    5400 4900
@@
 F 0 "RE15" H 5680 4854 50  0000 R CNN
 F 1 "18" H 5680 4945 50  0000 R CNN
-F 2 "Resistor_SMD:R_0805_2012Metric" V 5680 4900 50  0001 C CNN
+F 2 "Resistor_SMD:R_0603_1608Metric" V 5680 4900 50  0001 C CNN
 F 3 "~" H 5750 4900 50  0001 C CNN
 	1    5750 4900
@@
 F 0 "RC1" H 5530 1754 50  0000 R CNN
 F 1 "100" H 5530 1845 50  0000 R CNN
-F 2 "Resistor_SMD:R_0805_2012Metric" V 5530 1800 50  0001 C CNN
+F 2 "Resistor_SMD:R_0603_1608Metric" V 5530 1800 50  0001 C CNN
 F 3 "~" H 5600 1800 50  0001 C CNN
 	1    5600 1800
@@
 F 0 "CC3" H 6215 2496 50  0000 L CNN
 F 1 ".47u" H 6215 2405 50  0000 L CNN
-F 2 "Capacitor_SMD:C_0805_2012Metric" H 6138 2300 50  0001 C CNN
+F 2 "Capacitor_SMD:C_0603_1608Metric" H 6138 2300 50  0001 C CNN
 F 3 "~" H 6100 2450 50  0001 C CNN
 	1    6100 2450
@@
 F 0 "CC4" H 8515 1496 50  0000 L CNN
 F 1 ".47u" H 8515 1405 50  0000 L CNN
-F 2 "Capacitor_SMD:C_0805_2012Metric" H 8438 1300 50  0001 C CNN
+F 2 "Capacitor_SMD:C_0603_1608Metric" H 8438 1300 50  0001 C CNN
 F 3 "~" H 8400 1450 50  0001 C CNN
 	1    8400 1450
@@
 F 0 "RB2" H 6680 1754 50  0000 R CNN
 F 1 "9.1k" H 6680 1845 50  0000 R CNN
-F 2 "Resistor_SMD:R_0805_2012Metric" V 6680 1800 50  0001 C CNN
+F 2 "Resistor_SMD:R_0603_1608Metric" V 6680 1800 50  0001 C CNN
 F 3 "~" H 6750 1800 50  0001 C CNN
 	1    6750 1800
@@
 F 0 "Ri2" V 6850 2550 50  0000 R CNN
 F 1 "18" V 6950 2550 50  0000 R CNN
-F 2 "Resistor_SMD:R_0805_2012Metric" V 6980 2450 50  0001 C CNN
+F 2 "Resistor_SMD:R_0603_1608Metric" V 6980 2450 50  0001 C CNN
 F 3 "~" H 7050 2450 50  0001 C CNN
 	1    7050 2450
@@
 F 0 "Rsh2" H 7400 2750 50  0000 R CNN
 F 1 "120" H 7400 2650 50  0000 R CNN
-F 2 "Resistor_SMD:R_0805_2012Metric" V 7430 2700 50  0001 C CNN
+F 2 "Resistor_SMD:R_0603_1608Metric" V 7430 2700 50  0001 C CNN
 F 3 "~" H 7500 2700 50  0001 C CNN
 	1    7500 2700
@@
 F 0 "Csh2" H 7615 3296 50  0000 L CNN
 F 1 "1.2p" H 7615 3205 50  0000 L CNN
-F 2 "Capacitor_SMD:C_0805_2012Metric" H 7538 3100 50  0001 C CNN
+F 2 "Capacitor_SMD:C_0603_1608Metric" H 7538 3100 50  0001 C CNN
 F 3 "~" H 7500 3250 50  0001 C CNN
 	1    7500 3250
@@
 F 0 "RE21" H 8030 3204 50  0000 R CNN
 F 1 "150" H 8030 3295 50  0000 R CNN
-F 2 "Resistor_SMD:R_0805_2012Metric" V 8030 3250 50  0001 C CNN
+F 2 "Resistor_SMD:R_0603_1608Metric" V 8030 3250 50  0001 C CNN
 F 3 "~" H 8100 3250 50  0001 C CNN
 	1    8100 3250
@@
 F 0 "RE22" H 8430 3204 50  0000 R CNN
 F 1 "150" H 8430 3295 50  0000 R CNN
-F 2 "Resistor_SMD:R_0805_2012Metric" V 8430 3250 50  0001 C CNN
+F 2 "Resistor_SMD:R_0603_1608Metric" V 8430 3250 50  0001 C CNN
 F 3 "~" H 8500 3250 50  0001 C CNN
 	1    8500 3250
@@
 F 0 "Ro1" V 8800 2850 50  0000 R CNN
 F 1 "27" V 8900 2850 50  0000 R CNN
-F 2 "Resistor_SMD:R_0805_2012Metric" V 8930 2750 50  0001 C CNN
+F 2 "Resistor_SMD:R_0603_1608Metric" V 8930 2750 50  0001 C CNN
 F 3 "~" H 9000 2750 50  0001 C CNN
 	1    9000 2750
@@
 F 0 "CC5" H 9565 2796 50  0000 L CNN
 F 1 ".47u" H 9565 2705 50  0000 L CNN
-F 2 "Capacitor_SMD:C_0805_2012Metric" H 9488 2600 50  0001 C CNN
+F 2 "Capacitor_SMD:C_0603_1608Metric" H 9488 2600 50  0001 C CNN
 F 3 "~" H 9450 2750 50  0001 C CNN
 	1    9450 2750
@@
 	1    0    0    -1
 $EndComp
-$Comp
-L LNA_1-rescue:Barrel_Jack_MountingPin-Connector J3
-U 1 1 60111861
-P 1950 1500
-F 0 "J3" H 2007 1817 50  0000 C CNN
-F 1 "Barrel_Jack_MountingPin" H 2007 1726 50  0000 C CNN
-F 2 "Connector_BarrelJack:BarrelJack_Horizontal" H 2000 1460 50  0001 C CNN
-F 3 "~" H 2000 1460 50  0001 C CNN
-	1    1950 1500
-	1    0    0    -1
-$EndComp
-NoConn ~ 2250 1800
 $Comp
 L LNA_1-rescue:SMA-J-P-H-ST-EM1-RandomSMAIFoundOnline J1
@@
 	-1   0    0    1
 $EndComp
-Connection ~ 2700 1350
 Wire Wire Line
 	2250 1400 2600 1400
@@
 Wire Wire Line
 	2700 1650 2700 1800
-Connection ~ 2700 1650
 $Comp
 L LNA_1-rescue:SMA-J-P-H-ST-EM1-RandomSMAIFoundOnline J2
@@
 	-1   0    0    -1
 $EndComp
+Connection ~ 2700 1350
+Connection ~ 2700 1650
+$Comp
+L Connector_Generic:Conn_01x02 J3
+U 1 1 608FB524
+P 2050 1400
+F 0 "J3" H 1968 1617 50  0000 C CNN
+F 1 "Conn_01x02" H 1968 1526 50  0000 C CNN
+F 2 "Connector_PinSocket_2.00mm:PinSocket_1x02_P2.00mm_Vertical" H 2050 1400 50  0001 C CNN
+F 3 "~" H 2050 1400 50  0001 C CNN
+	1    2050 1400
+	-1   0    0    -1
+$EndComp
+Wire Wire Line
+	2250 1500 2250 1600
 $EndSCHEMATC
